Commit message: Backup COMPLETO: Scripts maestros y arreglos

File: tfg_ws/install/abb_irb140_support/share/abb_irb140_support/urdf/common_materials.xacro (robot description, xacro)
@@ -1,79 +1 @@
-<?xml version="1.0"?>
-<robot xmlns:xacro="http://ros.org/wiki/xacro">
-  <xacro:include filename="$(find abb_resources)/urdf/common_colours.xacro"/>
-  <xacro:macro name="material_abb_orange">
-    <material name="">
-      <color rgba="${colour_abb_orange}"/>
-    </material>
-  </xacro:macro>
-  <xacro:macro name="material_abb_graphite_white">
-    <material name="">
-      <color rgba="${colour_abb_graphite_white}"/>
-    </material>
-  </xacro:macro>
-  <xacro:macro name="material_abb_white">
-    <material name="">
-      <color rgba="${colour_abb_white}"/>
-    </material>
-  </xacro:macro>
-  <xacro:macro name="material_abb_pebble_gray">
-    <material name="">
-      <color rgba="${colour_abb_pebble_gray}"/>
-    </material>
-  </xacro:macro>
-  <xacro:macro name="material_abb_dark_gray">
-    <material name="">
-      <color rgba="${colour_abb_dark_gray}"/>
-    </material>
-  </xacro:macro>
-  <xacro:macro name="material_abb_black">
-    <material name="">
-      <color rgba="${colour_abb_black}"/>
-    </material>
-  </xacro:macro>
-  <xacro:macro name="material_abb_signal_red">
-    <material name="">
-      <color rgba="${colour_abb_signal_red}"/>
-    </material>
-  </xacro:macro>
-  <xacro:macro name="material_abb_carmine_red">
-    <material name="">
-      <color rgba="${colour_abb_carmine_red}"/>
-    </material>
-  </xacro:macro>
-  <xacro:macro name="material_abb_ultramarine_blue">
-    <material name="">
-      <color rgba="${colour_abb_ultramarine_blue}"/>
-    </material>
-  </xacro:macro>
-  <xacro:macro name="material_abb_sky_blue">
-    <material name="">
-      <color rgba="${colour_abb_sky_blue}"/>
-    </material>
-  </xacro:macro>
-  <xacro:macro name="material_abb_leaf_green">
-    <material name="">
-      <color rgba="${colour_abb_leaf_green}"/>
-    </material>
-  </xacro:macro>
-  <xacro:macro name="material_abb_olive_green">
-    <material name="">
-      <color rgba="${colour_abb_olive_green}"/>
-    </material>
-  </xacro:macro>
-  <xacro:macro name="material_abb_gray_white">
-    <material name="">
-      <color rgba="${colour_abb_gray_white}"/>
-    </material>
-  </xacro:macro>
-  <xacro:macro name="material_abb_pure_white">
-    <material name="">
-      <color rgba="${colour_abb_pure_white}"/>
-    </material>
-  </xacro:macro>
-  <xacro:macro name="material_abb_yellow">
-    <material name="">
-      <color rgba="${colour_abb_yellow}"/>
-    </material>
-  </xacro:macro>
-</robot>
+/home/ubuntu/tfg_ws/src/abb_irb140_support/urdf/common_materials.xacro

File: tfg_ws/install/abb_irb140_support/share/abb_irb140_support/urdf/irb140.xacro (robot description, xacro)
@@ -1,5 +1 @@
-<?xml version="1.0" ?>
-<robot name="abb_irb140" xmlns:xacro="http://ros.org/wiki/xacro">
-  <xacro:include filename="$(find abb_irb140_support)/urdf/irb140_macro.xacro"/>
-  <xacro:abb_irb140 prefix=""/>
-</robot>
+/home/ubuntu/tfg_ws/src/abb_irb140_support/urdf/irb140.xacro

File: tfg_ws/install/abb_irb140_support/share/abb_irb140_support/urdf/irb140_macro.xacro (robot description, xacro)
@@ -1,124 +1 @@
-<?xml version="1.0"?>
-<robot xmlns:xacro="http://ros.org/wiki/xacro">
-  <xacro:macro name="abb_irb140" params="prefix">
-    <link name="base_link">
-      <visual>
-        <origin xyz="0 0 0" rpy="0 0 0"/>
-        <geometry><mesh filename="package://abb_irb140_support/meshes/irb140/visual/base_link.stl"/></geometry>
-        <material name="abb_orange"><color rgba="1 0.43 0 1"/></material>
-      </visual>
-      <collision>
-        <origin xyz="0 0 0" rpy="0 0 0"/>
-        <geometry><mesh filename="package://abb_irb140_support/meshes/irb140/collision/base_link.stl"/></geometry>
-      </collision>
-    </link>
-    <link name="link_1">
-      <visual>
-        <origin xyz="0 0 0" rpy="0 0 0"/>
-        <geometry><mesh filename="package://abb_irb140_support/meshes/irb140/visual/link_1.stl"/></geometry>
-        <material name="abb_orange"/>
-      </visual>
-      <collision>
-        <origin xyz="0 0 0" rpy="0 0 0"/>
-        <geometry><mesh filename="package://abb_irb140_support/meshes/irb140/collision/link_1.stl"/></geometry>
-      </collision>
-    </link>
-    <link name="link_2">
-      <visual>
-        <origin xyz="0 0 0" rpy="0 0 0"/>
-        <geometry><mesh filename="package://abb_irb140_support/meshes/irb140/visual/link_2.stl"/></geometry>
-        <material name="abb_orange"/>
-      </visual>
-      <collision>
-        <origin xyz="0 0 0" rpy="0 0 0"/>
-        <geometry><mesh filename="package://abb_irb140_support/meshes/irb140/collision/link_2.stl"/></geometry>
-      </collision>
-    </link>
-    <link name="link_3">
-      <visual>
-        <origin xyz="0 0 0" rpy="0 0 0"/>
-        <geometry><mesh filename="package://abb_irb140_support/meshes/irb140/visual/link_3.stl"/></geometry>
-        <material name="abb_orange"/>
-      </visual>
-      <collision>
-        <origin xyz="0 0 0" rpy="0 0 0"/>
-        <geometry><mesh filename="package://abb_irb140_support/meshes/irb140/collision/link_3.stl"/></geometry>
-      </collision>
-    </link>
-    <link name="link_4">
-      <visual>
-        <origin xyz="0 0 0" rpy="0 0 0"/>
-        <geometry><mesh filename="package://abb_irb140_support/meshes/irb140/visual/link_4.stl"/></geometry>
-        <material name="abb_orange"/>
-      </visual>
-      <collision>
-        <origin xyz="0 0 0" rpy="0 0 0"/>
-        <geometry><mesh filename="package://abb_irb140_support/meshes/irb140/collision/link_4.stl"/></geometry>
-      </collision>
-    </link>
-    <link name="link_5">
-      <visual>
-        <origin xyz="0 0 0" rpy="0 0 0"/>
-        <geometry><mesh filename="package://abb_irb140_support/meshes/irb140/visual/link_5.stl"/></geometry>
-        <material name="abb_orange"/>
-      </visual>
-      <collision>
-        <origin xyz="0 0 0" rpy="0 0 0"/>
-        <geometry><mesh filename="package://abb_irb140_support/meshes/irb140/collision/link_5.stl"/></geometry>
-      </collision>
-    </link>
-    <link name="link_6">
-      <visual>
-        <origin xyz="0 0 0" rpy="0 0 0"/>
-        <geometry><mesh filename="package://abb_irb140_support/meshes/irb140/visual/link_6.stl"/></geometry>
-        <material name="abb_black"><color rgba="0 0 0 1"/></material>
-      </visual>
-      <collision>
-        <origin xyz="0 0 0" rpy="0 0 0"/>
-        <geometry><mesh filename="package://abb_irb140_support/meshes/irb140/collision/link_6.stl"/></geometry>
-      </collision>
-    </link>
-    <joint name="joint_1" type="revolute">
-      <origin xyz="0 0 0" rpy="0 0 0"/>
-      <parent link="base_link"/>
-      <child link="link_1"/>
-      <axis xyz="0 0 1"/>
-      <limit lower="-3.1416" upper="3.1416" effort="0" velocity="2.618"/>
-    </joint>
-    <joint name="joint_2" type="revolute">
-      <origin xyz="0.070 0 0.352" rpy="0 0 0"/>
-      <parent link="link_1"/>
-      <child link="link_2"/>
-      <axis xyz="0 1 0"/>
-      <limit lower="-1.5708" upper="1.9198" effort="0" velocity="2.618"/>
-    </joint>
-    <joint name="joint_3" type="revolute">
-      <origin xyz="0 -0.065 0.360" rpy="0 0 0"/>
-      <parent link="link_2"/>
-      <child link="link_3"/>
-      <axis xyz="0 1 0"/>
-      <limit lower="-4.0142" upper="0.8726" effort="0" velocity="2.618"/>
-    </joint>
-    <joint name="joint_4" type="revolute">
-      <origin xyz="0.239 0.065 0" rpy="0 0 0"/>
-      <parent link="link_3"/>
-      <child link="link_4"/>
-      <axis xyz="1 0 0"/>
-      <limit lower="-3.4906" upper="3.4906" effort="0" velocity="6.2832"/>
-    </joint>
-    <joint name="joint_5" type="revolute">
-      <origin xyz="0.141 0 0" rpy="0 0 0"/>
-      <parent link="link_4"/>
-      <child link="link_5"/>
-      <axis xyz="0 1 0"/>
-      <limit lower="-2.0071" upper="2.0071" effort="0" velocity="6.2832"/>
-    </joint>
-    <joint name="joint_6" type="revolute">
-      <origin xyz="0.065 0 0" rpy="0 0 0"/>
-      <parent link="link_5"/>
-      <child link="link_6"/>
-      <axis xyz="1 0 0"/>
-      <limit lower="-6.9813" upper="6.9813" effort="0" velocity="7.854"/>
-    </joint>
-  </xacro:macro>
-</robot>
+/home/ubuntu/tfg_ws/src/abb_irb140_support/urdf/irb140_macro.xacro
